Commit message: fix: load urdf with urdf string

File: example/objects/camera/assets/realsense2_d435.urdf (robot description, URDF)
Before this commit: robot realsense2_camera, 11 links, 10 joints
Links:
- link base_link: mass None -> 0.0
- link camera_bottom_screw_frame: mass None -> 0.0
- link camera_color_frame: mass None -> 0.0
- link camera_color_optical_frame: mass None -> 0.0
- link camera_depth_frame: mass None -> 0.0
- link camera_depth_optical_frame: mass None -> 0.0
- link camera_infra1_frame: mass None -> 0.0
- link camera_infra1_optical_frame: mass None -> 0.0
- link camera_infra2_frame: mass None -> 0.0
- link camera_infra2_optical_frame: mass None -> 0.0
